Commit message: Modified URDF file to reflect the real robot, and assembled the left wheel

File: ros2/src/mobile_robot/description/robot_core_old.xacro (robot description, xacro)
@@ -21,9 +21,11 @@
     </material>
     <!-- Chassis -->
+    <xacro:property name="chassis_length" value="0.33"/>
+    <xacro:property name="chassis_width" value="0.3"/>
     <xacro:property name="big_bar_length" value="0.3"/>
     <xacro:property name="chassis_thickness" value="0.015"/>
-    <xacro:property name="front_base_length" value="0.2"/>
-    <xacro:property name="base_to_back_distance" value="0.05"/>
-    <xacro:property name="a" value="0.08"/>
+    <xacro:property name="front_base_length" value="0.05"/>
+    <xacro:property name="back_base_length" value="0.05"/>
+    <xacro:property name="a" value="0.02"/>
 	<!-- Create fixed world frame -->
 	<link name="world"></link>
@@ -39,5 +41,5 @@
             </geometry>
             <material name="orange"/>
-            <origin xyz="0 ${-base_to_back_distance - chassis_thickness/2} 0"/>
+            <origin xyz="0 ${-big_bar_length/2 +chassis_thickness/2} 0"/>
         </visual>
         <visual>
@@ -45,5 +47,5 @@
                 <box size="${big_bar_length} ${chassis_thickness} ${chassis_thickness}"/>
             </geometry>
-            <origin xyz="0 ${big_bar_length - base_to_back_distance + chassis_thickness/2} 0"/>
+            <origin xyz="0 ${big_bar_length/2 -chassis_thickness/2} 0"/>
         </visual>
         <visual>
@@ -52,5 +54,5 @@
             </geometry>
             <material name="grey"/>
-            <origin xyz="${-big_bar_length/2+chassis_thickness/2} ${big_bar_length/2 - base_to_back_distance} 0"/>
+            <origin xyz="${-big_bar_length/2 - chassis_thickness/2} 0 0"/>
         </visual>
         <visual>
@@ -59,17 +61,17 @@
             </geometry>
             <material name="grey"/>
-            <origin xyz="${big_bar_length/2-chassis_thickness/2} ${big_bar_length/2 - base_to_back_distance} 0"/>
-        </visual>
-        <visual>
-            <geometry>
-                <box size="${big_bar_length} ${chassis_thickness} ${chassis_thickness}"/>
-            </geometry>
-            <origin xyz="0 0 ${chassis_thickness}"/>
-        </visual>
-        <visual>
-            <geometry>
-                <box size="${big_bar_length} ${chassis_thickness} ${chassis_thickness}"/>
-            </geometry>
-            <origin xyz="0 ${front_base_length} ${chassis_thickness}"/>
+            <origin xyz="${big_bar_length/2 + chassis_thickness/2} 0 0"/>
+        </visual>
+        <visual>
+            <geometry>
+                <box size="${chassis_thickness} ${big_bar_length} ${chassis_thickness}"/>
+            </geometry>
+            <origin xyz="${front_base_length} 0 ${chassis_thickness}"/>
+        </visual>
+        <visual>
+            <geometry>
+                <box size="${chassis_thickness} ${chassis_width} ${chassis_thickness}"/>
+            </geometry>
+            <origin xyz="${-back_base_length} 0 ${chassis_thickness}"/>
         </visual>
         <inertial>
@@ -81,39 +83,38 @@
 		<material>Gazebo/White</material>
     </gazebo>
-    <xacro:property name="a" value="0.08"/>
-    <xacro:property name="l1" value="0.05"/>
-    <xacro:property name="l2" value="0.017"/>
-    <xacro:property name="l3" value="0.076"/>
+    <xacro:property name="l1" value="0.1"/>
+    <xacro:property name="l2" value="0.04"/>
+    <xacro:property name="l3" value="0.033"/>
     <xacro:property name="thickness" value="0.015"/>
     <xacro:property name="motor_side" value="0.02"/>
-    <xacro:property name="wheel_thickness" value="0.01"/>
-    <xacro:property name="l4" value="${l2-thickness/2-wheel_thickness/2}"/>
-    <xacro:property name="l_tot" value="${l1+l3+thickness}"/>
     <!-- Left_wheel_base-->
     <link name="left_wheel_base">
         <visual>
             <geometry>
-                <box size="${thickness} ${thickness} ${l1}" />
-            </geometry>
-            <origin xyz="${-a} 0 ${-l1/2+thickness/2}"/>
+                <box size="${l1} ${thickness} ${thickness}" />
+            </geometry>
+            <origin xyz="${-l1/2} 0 0"/>
             <material name="white"/>
         </visual>
-        <visual>
-            <geometry>
-                <box size="${l2} ${thickness} ${thickness}"/>
-            </geometry>
-            <origin xyz="${-a-l2/2-thickness/2} 0 ${-l1+thickness}"/>
-        </visual>
-        <visual>
-            <geometry>
-                <box size="${thickness} ${thickness} ${l3}"/>
-            </geometry>
-            <origin xyz="${-a-l2} ${0} ${-l3/2-l1+thickness/2}"/>
-        </visual>
-        <visual>
-            <geometry>
-                <box size="${l4} ${thickness} ${thickness}"/>
-            </geometry>
-            <origin xyz="${-a-wheel_thickness/2-l4/2} 0 ${-l_tot+2*thickness}"/>
+        <xacro:inertial_box mass="0.5" x="0.3" y="0.3" z="0.15">
+			<origin xyz="0 ${-chassis_width/2 +chassis_thickness/2} 0" rpy="0 0 0"/>
+        </xacro:inertial_box>
+        <visual>
+            <geometry>
+                <box size="${thickness} ${l2} ${thickness}"/>
+            </geometry>
+            <origin xyz="${-l1+thickness/2} ${-l2/2-thickness/2} 0.0" rpy="0.0 0.0 0.0"/>
+        </visual>
+        <visual>
+            <geometry>
+                <box size="${l3} ${thickness} ${thickness}"/>
+            </geometry>
+            <origin xyz="${-l1-l3/2} ${-l2} 0.0" rpy="0.0 0.0 0.0"/>
+        </visual>
+        <visual>
+            <geometry>
+                <box size="${motor_side} ${motor_side} ${motor_side}"/>
+            </geometry>
+            <origin xyz="${-l1-l3-motor_side/2} ${-l2} 0.0" rpy="0.0 0.0 0.0"/>
         </visual>
         <inertial>
@@ -128,14 +129,22 @@
         <parent link="chassis"/>
         <child link="left_wheel_base"/>
-        <origin xyz="${0} ${0} ${0}" rpy="0.0 0.0 0.0"/>
+        <origin xyz="${front_base_length} ${chassis_width/2-a} ${chassis_thickness/2}" rpy="0.0 ${-pi/2} 0.0"/>
     </joint>
     <!-- Left_wheel-->
     <xacro:property name="wheel_radius" value="0.033"/>
+    <xacro:property name="wheel_length" value="0.02"/>
     <link name="left_wheel">
         <visual>
             <geometry>
-                <cylinder radius="${wheel_radius}" length="${wheel_thickness}"/>
-            </geometry>
-            <origin xyz="${-a} 0 ${-l_tot+wheel_radius}" rpy="0 ${-pi/2} 0"/>
+                <box size="${thickness} ${l2-wheel_length/2-motor_side/2} ${thickness}"/>
+            </geometry>
+            <origin xyz="0 ${-(l2-wheel_length/2-motor_side/2+wheel_length)/2} 0"/>
+			<material name="grey"/>
+        </visual>
+        <visual>
+            <geometry>
+                <cylinder radius="${wheel_radius}" length="${wheel_length}"/>
+            </geometry>
+            <origin xyz="0 0 0.0" rpy="${pi/2} 0.0 0.0"/>
 			<material name="grey"/>
         </visual>
@@ -144,5 +153,5 @@
         <parent link="left_wheel_base"/>
         <child link="left_wheel"/>
-        <origin xyz="0 0 0"/>
+        <origin xyz="${-l1-l3-motor_side/2} ${0} 0"/>
         <axis xyz="0 1 0"/>
     </joint>
@@ -151,26 +160,29 @@
         <visual>
             <geometry>
-                <box size="${thickness} ${thickness} ${l1}" />
-            </geometry>
-            <origin xyz="${a} 0 ${-l1/2+thickness/2}"/>
+                <box size="${l1} ${thickness} ${thickness}" />
+            </geometry>
+            <origin xyz="${-l1/2} 0 0"/>
             <material name="white"/>
         </visual>
-        <visual>
-            <geometry>
-                <box size="${l2} ${thickness} ${thickness}"/>
-            </geometry>
-            <origin xyz="${a} 0 ${-l1-thickness/2}"/>
-        </visual>
-        <visual>
-            <geometry>
-                <box size="${thickness} ${thickness} ${l3}"/>
-            </geometry>
-            <origin xyz="${a+l2+thickness/2} ${-l3/2} 0.0"/>
-        </visual>
-        <visual>
-            <geometry>
-                <box size="${l4} ${thickness} ${thickness}"/>
-            </geometry>
-            <origin xyz="${l4/2} 0 ${-l_tot}"/>
+        <xacro:inertial_box mass="0.5" x="0.3" y="0.3" z="0.15">
+			<origin xyz="0 ${-chassis_width/2 +chassis_thickness/2} 0" rpy="0 0 0"/>
+        </xacro:inertial_box>
+        <visual>
+            <geometry>
+                <box size="${thickness} ${l2} ${thickness}"/>
+            </geometry>
+            <origin xyz="${-l1+thickness/2} ${-l2/2-thickness/2} 0.0" rpy="0.0 0.0 0.0"/>
+        </visual>
+        <visual>
+            <geometry>
+                <box size="${l3} ${thickness} ${thickness}"/>
+            </geometry>
+            <origin xyz="${-l1-l3/2} ${-l2} 0.0" rpy="0.0 0.0 0.0"/>
+        </visual>
+        <visual>
+            <geometry>
+                <box size="${motor_side} ${motor_side} ${motor_side}"/>
+            </geometry>
+            <origin xyz="${-l1-l3-motor_side/2} ${-l2} 0.0" rpy="0.0 0.0 0.0"/>
         </visual>
         <inertial>
@@ -185,5 +197,5 @@
         <parent link="chassis"/>
         <child link="right_wheel_base"/>
-        <origin xyz="${a} ${0} ${-thickness/2}" rpy="0.0 0.0 0.0"/>
+        <origin xyz="${front_base_length} ${-chassis_width/2+a} ${chassis_thickness/2}" rpy="0.0 ${-pi/2} ${pi}"/>
     </joint>
     <!-- right_wheel-->
@@ -191,9 +203,20 @@
         <visual>
             <geometry>
-                <cylinder radius="${wheel_radius}" length="${wheel_thickness}"/>
-            </geometry>
-            <origin xyz="0 0 0.0" rpy="0 0.0 ${pi/2}"/>
-			<material name="grey"/>
-        </visual>
+                <box size="${thickness} ${l2-wheel_length/2-motor_side/2} ${thickness}"/>
+            </geometry>
+            <origin xyz="0 ${-(l2-wheel_length/2-motor_side/2+wheel_length)/2} 0"/>
+            <material name="grey"/>
+        </visual>
+        <visual>
+            <geometry>
+                <cylinder radius="${wheel_radius}" length="${wheel_length}"/>
+            </geometry>
+            <origin xyz="0 0 0.0" rpy="${pi/2} 0.0 0.0"/>
+            <material name="grey"/>
+        </visual>
+        <inertial>
+			<mass value="1"/>
+			<inertia ixx="1e-3" ixy="0.0" ixz="0.0" iyy="1e-3" iyz="0.0" izz="1e-3"/>
+		</inertial>
     </link>
     <gazebo reference="right_wheel">
@@ -203,5 +226,5 @@
         <parent link="right_wheel_base"/>
         <child link="right_wheel"/>
-        <origin xyz="0 0 ${-l1-l3-wheel_radius}"/>
+        <origin xyz="${-l1-l3-motor_side/2} ${0} 0"/>
         <axis xyz="0 1 0"/>
     </joint>
@@ -210,5 +233,5 @@
 		<visual>
 			<geometry>
-				<box size="${thickness} ${thickness} ${l1+l3+thickness}"/>
+				<box size="${thickness} ${thickness} ${l1+l3+2*thickness}"/>
 			</geometry>
 			<material name="white"/>
@@ -218,5 +241,5 @@
 				<sphere radius="${wheel_radius}"/>
 			</geometry>
-			<origin xyz="0 0 ${-(l1+l3+wheel_radius)}"/>
+			<origin xyz="0 0 ${-(l1+l3)/2}"/>
 		</visual>
     </link>
@@ -224,5 +247,5 @@
 		<parent link="chassis"></parent>
 		<child link="castor_wheel"></child>
-        <origin xyz="0 ${front_base_length} ${-(l1+l3+wheel_radius)}" />
+        <origin xyz="${-front_base_length} 0 ${-(l1+l3)/2}" />
 	</joint>
 </robot>

Commit message: Finished detailing robot model, added new function in sim.cpp to determine the ICR at all times and publish it to /tf

File: ros2/src/mobile_robot/description/robot_core_old.xacro (robot description, xacro)
@@ -21,8 +21,7 @@
     </material>
     <!-- Chassis -->
-    <xacro:property name="chassis_length" value="0.33"/>
-    <xacro:property name="chassis_width" value="0.3"/>
-    <xacro:property name="big_bar_length" value="0.3"/>
-    <xacro:property name="chassis_thickness" value="0.015"/>
+    <xacro:property name="chassis_length" value="0.2"/>
+    <xacro:property name="chassis_width" value="0.1"/>
+    <xacro:property name="chassis_thickness" value="0.01"/>
     <xacro:property name="front_base_length" value="0.05"/>
     <xacro:property name="back_base_length" value="0.05"/>
@@ -38,32 +37,32 @@
 		<visual>
             <geometry>
-                <box size="${big_bar_length} ${chassis_thickness} ${chassis_thickness}"/>
+                <box size="${chassis_length} ${chassis_thickness} ${chassis_thickness}"/>
             </geometry>
             <material name="orange"/>
-            <origin xyz="0 ${-big_bar_length/2 +chassis_thickness/2} 0"/>
-        </visual>
-        <visual>
-            <geometry>
-                <box size="${big_bar_length} ${chassis_thickness} ${chassis_thickness}"/>
-            </geometry>
-            <origin xyz="0 ${big_bar_length/2 -chassis_thickness/2} 0"/>
-        </visual>
-        <visual>
-            <geometry>
-                <box size="${chassis_thickness} ${big_bar_length} ${chassis_thickness}"/>
-            </geometry>
-            <material name="grey"/>
-            <origin xyz="${-big_bar_length/2 - chassis_thickness/2} 0 0"/>
-        </visual>
-        <visual>
-            <geometry>
-                <box size="${chassis_thickness} ${big_bar_length} ${chassis_thickness}"/>
-            </geometry>
-            <material name="grey"/>
-            <origin xyz="${big_bar_length/2 + chassis_thickness/2} 0 0"/>
-        </visual>
-        <visual>
-            <geometry>
-                <box size="${chassis_thickness} ${big_bar_length} ${chassis_thickness}"/>
+            <origin xyz="0 ${-chassis_width/2 +chassis_thickness/2} 0"/>
+        </visual>
+        <visual>
+            <geometry>
+                <box size="${chassis_length} ${chassis_thickness} ${chassis_thickness}"/>
+            </geometry>
+            <origin xyz="0 ${chassis_width/2 -chassis_thickness/2} 0"/>
+        </visual>
+        <visual>
+            <geometry>
+                <box size="${chassis_thickness} ${chassis_width} ${chassis_thickness}"/>
+            </geometry>
+            <material name="grey"/>
+            <origin xyz="${-chassis_length/2} 0 0"/>
+        </visual>
+        <visual>
+            <geometry>
+                <box size="${chassis_thickness} ${chassis_width} ${chassis_thickness}"/>
+            </geometry>
+            <material name="grey"/>
+            <origin xyz="${chassis_length/2} 0 0"/>
+        </visual>
+        <visual>
+            <geometry>
+                <box size="${chassis_thickness} ${chassis_width} ${chassis_thickness}"/>
             </geometry>
             <origin xyz="${front_base_length} 0 ${chassis_thickness}"/>
@@ -83,8 +82,8 @@
 		<material>Gazebo/White</material>
     </gazebo>
-    <xacro:property name="l1" value="0.1"/>
-    <xacro:property name="l2" value="0.04"/>
-    <xacro:property name="l3" value="0.033"/>
-    <xacro:property name="thickness" value="0.015"/>
+    <xacro:property name="l1" value="0.04"/>
+    <xacro:property name="l2" value="0.01"/>
+    <xacro:property name="l3" value="0.025"/>
+    <xacro:property name="thickness" value="0.01"/>
     <xacro:property name="motor_side" value="0.02"/>
     <!-- Left_wheel_base-->
@@ -132,6 +131,6 @@
     </joint>
     <!-- Left_wheel-->
-    <xacro:property name="wheel_radius" value="0.033"/>
-    <xacro:property name="wheel_length" value="0.02"/>
+    <xacro:property name="wheel_radius" value="0.025"/>
+    <xacro:property name="wheel_length" value="0.01"/>
     <link name="left_wheel">
         <visual>
@@ -233,5 +232,5 @@
 		<visual>
 			<geometry>
-				<box size="${thickness} ${thickness} ${l1+l3+2*thickness}"/>
+				<box size="${thickness} ${thickness} ${l1+l3}"/>
 			</geometry>
 			<material name="white"/>
@@ -241,5 +240,5 @@
 				<sphere radius="${wheel_radius}"/>
 			</geometry>
-			<origin xyz="0 0 ${-(l1+l3)/2}"/>
+			<origin xyz="0 0 ${-(l1+l3)/2-wheel_radius+motor_side/4}"/>
 		</visual>
     </link>
@@ -247,5 +246,5 @@
 		<parent link="chassis"></parent>
 		<child link="castor_wheel"></child>
-        <origin xyz="${-front_base_length} 0 ${-(l1+l3)/2}" />
+        <origin xyz="${-front_base_length} 0 ${-2*chassis_thickness}" />
 	</joint>
 </robot>
