Commit message: Created launch file for simulation, corrected come URDF parameters and added a transform for the ICR.

File: ros2/src/mobile_robot/description/robot_core.xacro (robot description, xacro)
@@ -21,7 +21,7 @@
     </material>
     <!-- Chassis -->
-    <xacro:property name="chassis_length" value="0.2"/>
-    <xacro:property name="chassis_width" value="0.1"/>
-    <xacro:property name="chassis_thickness" value="0.01"/>
+    <xacro:property name="chassis_length" value="0.33"/>
+    <xacro:property name="chassis_width" value="0.3"/>
+    <xacro:property name="chassis_thickness" value="0.015"/>
     <xacro:property name="front_base_length" value="0.05"/>
     <xacro:property name="back_base_length" value="0.05"/>
@@ -82,8 +82,8 @@
 		<material>Gazebo/White</material>
     </gazebo>
-    <xacro:property name="l1" value="0.04"/>
-    <xacro:property name="l2" value="0.01"/>
-    <xacro:property name="l3" value="0.025"/>
-    <xacro:property name="thickness" value="0.01"/>
+    <xacro:property name="l1" value="0.1"/>
+    <xacro:property name="l2" value="0.04"/>
+    <xacro:property name="l3" value="0.033"/>
+    <xacro:property name="thickness" value="0.015"/>
     <xacro:property name="motor_side" value="0.02"/>
     <!-- Left_wheel_base-->
@@ -131,6 +131,6 @@
     </joint>
     <!-- Left_wheel-->
-    <xacro:property name="wheel_radius" value="0.025"/>
-    <xacro:property name="wheel_length" value="0.01"/>
+    <xacro:property name="wheel_radius" value="0.033"/>
+    <xacro:property name="wheel_length" value="0.02"/>
     <link name="left_wheel">
         <visual>
@@ -232,5 +232,5 @@
 		<visual>
 			<geometry>
-				<box size="${thickness} ${thickness} ${l1+l3}"/>
+				<box size="${thickness} ${thickness} ${l1+l3+2*thickness}"/>
 			</geometry>
 			<material name="white"/>
@@ -240,5 +240,5 @@
 				<sphere radius="${wheel_radius}"/>
 			</geometry>
-			<origin xyz="0 0 ${-(l1+l3)/2-wheel_radius+motor_side/4}"/>
+			<origin xyz="0 0 ${-(l1+l3)/2}"/>
 		</visual>
     </link>
@@ -246,5 +246,5 @@
 		<parent link="chassis"></parent>
 		<child link="castor_wheel"></child>
-        <origin xyz="${-front_base_length} 0 ${-2*chassis_thickness}" />
+        <origin xyz="${-front_base_length} 0 ${-(l1+l3)/2}" />
 	</joint>
 </robot>

Commit message: Finished URDF assembly and modified sim.cpp to send beta2=d2+M_PI

File: ros2/src/mobile_robot/description/robot_core.xacro (robot description, xacro)
@@ -96,5 +96,5 @@
                 <box size="${thickness} ${thickness} ${l1}" />
             </geometry>
-            <origin xyz="${-a} 0 ${-l1/2+thickness/2}"/>
+            <origin xyz="${0} 0 ${-l1/2}"/>
             <material name="white"/>
         </visual>
@@ -103,5 +103,5 @@
                 <box size="${l2} ${thickness} ${thickness}"/>
             </geometry>
-            <origin xyz="${-a-l2/2-thickness/2} 0 ${-l1+thickness}"/>
+            <origin xyz="${-l2/2-thickness/2} 0 ${-l1+thickness/2}"/>
         </visual>
         <visual>
@@ -109,5 +109,5 @@
                 <box size="${thickness} ${thickness} ${l3}"/>
             </geometry>
-            <origin xyz="${-a-l2} ${0} ${-l3/2-l1+thickness/2}"/>
+            <origin xyz="${-l2} ${0} ${-l3/2-l1}"/>
         </visual>
         <visual>
@@ -115,5 +115,5 @@
                 <box size="${l4} ${thickness} ${thickness}"/>
             </geometry>
-            <origin xyz="${-a-wheel_thickness/2-l4/2} 0 ${-l_tot+2*thickness}"/>
+            <origin xyz="${-wheel_thickness/2-l4/2} 0 ${-l_tot+3*thickness/2}"/>
         </visual>
         <inertial>
@@ -128,5 +128,6 @@
         <parent link="chassis"/>
         <child link="left_wheel_base"/>
-        <origin xyz="${0} ${0} ${0}" rpy="0.0 0.0 0.0"/>
+        <origin xyz="${-a} ${0} ${thickness/2}" rpy="0.0 0.0 ${pi/2}"/>
+        <axis xyz="0 0 1"/>
     </joint>
     <!-- Left_wheel-->
@@ -137,5 +138,5 @@
                 <cylinder radius="${wheel_radius}" length="${wheel_thickness}"/>
             </geometry>
-            <origin xyz="${-a} 0 ${-l_tot+wheel_radius}" rpy="0 ${-pi/2} 0"/>
+            <origin xyz="${0} 0 ${0}" rpy="${pi/2} 0 0"/>
 			<material name="grey"/>
         </visual>
@@ -144,14 +145,14 @@
         <parent link="left_wheel_base"/>
         <child link="left_wheel"/>
-        <origin xyz="0 0 0"/>
+        <origin xyz="${0} 0 ${-l_tot-thickness+wheel_radius}" rpy="0 0 ${pi/2}"/>
         <axis xyz="0 1 0"/>
     </joint>
     <!-- right_wheel_base-->
     <link name="right_wheel_base">
-        <visual>
+<visual>
             <geometry>
                 <box size="${thickness} ${thickness} ${l1}" />
             </geometry>
-            <origin xyz="${a} 0 ${-l1/2+thickness/2}"/>
+            <origin xyz="${0} 0 ${-l1/2}"/>
             <material name="white"/>
         </visual>
@@ -160,5 +161,5 @@
                 <box size="${l2} ${thickness} ${thickness}"/>
             </geometry>
-            <origin xyz="${a} 0 ${-l1-thickness/2}"/>
+            <origin xyz="${-l2/2-thickness/2} 0 ${-l1+thickness/2}"/>
         </visual>
         <visual>
@@ -166,5 +167,5 @@
                 <box size="${thickness} ${thickness} ${l3}"/>
             </geometry>
-            <origin xyz="${a+l2+thickness/2} ${-l3/2} 0.0"/>
+            <origin xyz="${-l2} ${0} ${-l3/2-l1}"/>
         </visual>
         <visual>
@@ -172,5 +173,5 @@
                 <box size="${l4} ${thickness} ${thickness}"/>
             </geometry>
-            <origin xyz="${l4/2} 0 ${-l_tot}"/>
+            <origin xyz="${-wheel_thickness/2-l4/2} 0 ${-l_tot+3*thickness/2}"/>
         </visual>
         <inertial>
@@ -185,5 +186,6 @@
         <parent link="chassis"/>
         <child link="right_wheel_base"/>
-        <origin xyz="${a} ${0} ${-thickness/2}" rpy="0.0 0.0 0.0"/>
+        <origin xyz="${a} ${0} ${thickness/2}" rpy="0.0 0.0 ${-pi/2}"/>
+        <axis xyz="0 0 1"/>
     </joint>
     <!-- right_wheel-->
@@ -193,5 +195,5 @@
                 <cylinder radius="${wheel_radius}" length="${wheel_thickness}"/>
             </geometry>
-            <origin xyz="0 0 0.0" rpy="0 0.0 ${pi/2}"/>
+            <origin xyz="${0} 0 ${0}" rpy="${pi/2} 0 0"/>
 			<material name="grey"/>
         </visual>
@@ -203,5 +205,5 @@
         <parent link="right_wheel_base"/>
         <child link="right_wheel"/>
-        <origin xyz="0 0 ${-l1-l3-wheel_radius}"/>
+        <origin xyz="${0} 0 ${-l_tot-thickness+wheel_radius}" rpy="0 0 ${pi/2}"/>
         <axis xyz="0 1 0"/>
     </joint>
@@ -210,6 +212,7 @@
 		<visual>
 			<geometry>
-				<box size="${thickness} ${thickness} ${l1+l3+thickness}"/>
+				<box size="${thickness} ${thickness} ${l1+l3}"/>
 			</geometry>
+            <origin xyz="0 0 ${-(l1+l3)/2}"/>
 			<material name="white"/>
 		</visual>
@@ -218,5 +221,5 @@
 				<sphere radius="${wheel_radius}"/>
 			</geometry>
-			<origin xyz="0 0 ${-(l1+l3+wheel_radius)}"/>
+			<origin xyz="0 0 ${-(l1+l3)}"/>
 		</visual>
     </link>
@@ -224,5 +227,5 @@
 		<parent link="chassis"></parent>
 		<child link="castor_wheel"></child>
-        <origin xyz="0 ${front_base_length} ${-(l1+l3+wheel_radius)}" />
+        <origin xyz="0 ${front_base_length} ${thickness/2}" />
 	</joint>
 </robot>

Commit message: Added QDoubleSpinboxes to all the sliders to have a visual aid while setting values in the GUI. Added a validation in sim.cpp for when the difference between angles is 0. This caused the ICR to be located at infinity and rviz would crash when showing the frame.

File: ros2/src/mobile_robot/description/robot_core.xacro (robot description, xacro)
@@ -73,8 +73,4 @@
             <origin xyz="0 ${front_base_length} ${chassis_thickness}"/>
         </visual>
-        <inertial>
-			<mass value="1"/>
-			<inertia ixx="1e-3" ixy="0.0" ixz="0.0" iyy="1e-3" iyz="0.0" izz="1e-3"/>
-		</inertial>
     </link>
     <gazebo reference="chassis">
@@ -117,8 +113,4 @@
             <origin xyz="${-wheel_thickness/2-l4/2} 0 ${-l_tot+3*thickness/2}"/>
         </visual>
-        <inertial>
-			<mass value="1"/>
-			<inertia ixx="1e-3" ixy="0.0" ixz="0.0" iyy="1e-3" iyz="0.0" izz="1e-3"/>
-		</inertial>
     </link>
     <gazebo reference="left_wheel_base_joint">
@@ -175,8 +167,4 @@
             <origin xyz="${-wheel_thickness/2-l4/2} 0 ${-l_tot+3*thickness/2}"/>
         </visual>
-        <inertial>
-			<mass value="1"/>
-			<inertia ixx="1e-3" ixy="0.0" ixz="0.0" iyy="1e-3" iyz="0.0" izz="1e-3"/>
-		</inertial>
     </link>
     <gazebo reference="right_wheel_base_joint">

Commit message: Restricted GUI to only be able to choose one mode each launch. Also changed the way the mode is notified to the node. Previously it was published in a topic, now it's passed as an argument when the user presses "launch"

File: ros2/src/mobile_robot/description/robot_core.xacro (robot description, xacro)
@@ -23,6 +23,6 @@
     <xacro:property name="big_bar_length" value="0.3"/>
     <xacro:property name="chassis_thickness" value="0.015"/>
-    <xacro:property name="front_base_length" value="0.2"/>
-    <xacro:property name="base_to_back_distance" value="0.05"/>
+    <xacro:property name="front_base_length" value="0.18"/>
+    <xacro:property name="base_to_back_distance" value="0.065"/>
     <xacro:property name="a" value="0.08"/>
 	<!-- Create fixed world frame -->
