Commit message: Added two more fields to the position command message. Changed the way in which we are sending the commands to the motor_cmd topic (removed mode field)

File: ros2/src/workstation/description/robot_core.xacro (robot description, xacro)
@@ -20,5 +20,5 @@
         <color rgba="0.5 0.5 0.5 1"/>
     </material>
-    <!-- Chassis -->
+    <!-- base_link -->
     <xacro:property name="big_bar_length" value="0.3"/>
     <xacro:property name="chassis_thickness" value="0.015"/>
@@ -26,12 +26,12 @@
     <xacro:property name="base_to_back_distance" value="0.065"/>
     <xacro:property name="a" value="0.08"/>
-	<!-- Create fixed world frame -->
-	<link name="world"></link>
+	<!-- Create fixed odom frame -->
+	<link name="odom"></link>
 	<joint name="world_joint" type="floating">
-		<parent link="world"></parent>
-		<child link="chassis"></child>
+		<parent link="odom"></parent>
+		<child link="base_link"></child>
 		<origin xyz="0 0 0.1"></origin>
 	</joint>
-    <link name="chassis">
+    <link name="base_link">
 		<visual>
             <geometry>
@@ -74,5 +74,5 @@
         </visual>
     </link>
-    <gazebo reference="chassis">
+    <gazebo reference="base_link">
 		<material>Gazebo/White</material>
     </gazebo>
@@ -99,5 +99,5 @@
                 <box size="${l2} ${thickness} ${thickness}"/>
             </geometry>
-            <origin xyz="${-l2/2-thickness/2} 0 ${-l1+thickness/2}"/>
+            <origin xyz="${l2/2+thickness/2} 0 ${-l1+thickness/2}"/>
         </visual>
         <visual>
@@ -105,5 +105,5 @@
                 <box size="${thickness} ${thickness} ${l3}"/>
             </geometry>
-            <origin xyz="${-l2} ${0} ${-l3/2-l1}"/>
+            <origin xyz="${l2} ${0} ${-l3/2-l1}"/>
         </visual>
         <visual>
@@ -111,5 +111,5 @@
                 <box size="${l4} ${thickness} ${thickness}"/>
             </geometry>
-            <origin xyz="${-wheel_thickness/2-l4/2} 0 ${-l_tot+3*thickness/2}"/>
+            <origin xyz="${wheel_thickness/2+l4/2} 0 ${-l_tot+3*thickness/2}"/>
         </visual>
     </link>
@@ -118,5 +118,5 @@
     </gazebo>
     <joint name="left_wheel_base_joint" type="continuous">
-        <parent link="chassis"/>
+        <parent link="base_link"/>
         <child link="left_wheel_base"/>
         <origin xyz="${-a} ${0} ${thickness/2}" rpy="0.0 0.0 ${pi/2}"/>
@@ -153,5 +153,5 @@
                 <box size="${l2} ${thickness} ${thickness}"/>
             </geometry>
-            <origin xyz="${-l2/2-thickness/2} 0 ${-l1+thickness/2}"/>
+            <origin xyz="${l2/2+thickness/2} 0 ${-l1+thickness/2}"/>
         </visual>
         <visual>
@@ -159,5 +159,5 @@
                 <box size="${thickness} ${thickness} ${l3}"/>
             </geometry>
-            <origin xyz="${-l2} ${0} ${-l3/2-l1}"/>
+            <origin xyz="${l2} ${0} ${-l3/2-l1}"/>
         </visual>
         <visual>
@@ -165,5 +165,5 @@
                 <box size="${l4} ${thickness} ${thickness}"/>
             </geometry>
-            <origin xyz="${-wheel_thickness/2-l4/2} 0 ${-l_tot+3*thickness/2}"/>
+            <origin xyz="${wheel_thickness/2+l4/2} 0 ${-l_tot+3*thickness/2}"/>
         </visual>
     </link>
@@ -172,5 +172,5 @@
     </gazebo>
     <joint name="right_wheel_base_joint" type="continuous">
-        <parent link="chassis"/>
+        <parent link="base_link"/>
         <child link="right_wheel_base"/>
         <origin xyz="${a} ${0} ${thickness/2}" rpy="0.0 0.0 ${-pi/2}"/>
@@ -213,5 +213,5 @@
     </link>
 	<joint name="castor_joint" type="fixed">
-		<parent link="chassis"></parent>
+		<parent link="base_link"></parent>
 		<child link="castor_wheel"></child>
         <origin xyz="0 ${front_base_length} ${thickness/2}" />
